File: BluetoothBlinker-PCB/BluetoothBlinker-PCB.kicad_pcb (KiCad board)
At the start: 2 copper layers, 73.9 x 37.3 mm, 51 parts, among them J1 USB_C_Receptacle_USB2.0, J2 Programming Connector, J3 Expansion Header, SW1 SW_Push, U1 CH340C, U2 TLV75533PDBV, U3 CC2642R, Y1 48MHz, Y2 32.768kHz

Commit message: Update to new USB Uart and generate PDF
Parts:
- U1: value CH340C -> CH340E; footprint Package_SO:SOIC-16_3.9x9.9mm_P1.27mm -> Package_SO:MSOP-10_3x3mm_P0.5mm
- moved U1 2.54 mm to (176.5, -17.5), turned to 270 degrees
Connections:
- AE1 pad 2: GND -> (no net)
- U1 pad 1: GND -> /D+
- U1 pad 10: Net-(U1-Pad10) -> /VDD
- U1 pad 2: /DEBUG_TX_MCU -> /D-
- U1 pad 3: /DEBUG_RX_MCU -> GND
- U1 pad 4: /VDD -> /DEBUG_DTR_MCU
- U1 pad 5: /D+ -> /DEBUG_CTS_MCU
- U1 pad 6: /D- -> Net-(U1-Pad6)
- U1 pad 7: Net-(U1-Pad7) -> /VDD
- U1 pad 8: Net-(U1-Pad8) -> /DEBUG_TX_MCU
- U1 pad 9: /DEBUG_CTS_MCU -> /DEBUG_RX_MCU
- U3 pad 30: /DEBUG_RX_MCU -> /DEBUG_TX_MCU
- U3 pad 31: /DEBUG_TX_MCU -> /DEBUG_RX_MCU
Routing:
- net /DEBUG_DTR_MCU: track 23.4 -> 15.3 mm
- net /D+: track 18.4 -> 20.6 mm
- net /D-: track 18.1 -> 20.1 mm
- net /DEBUG_CTS_MCU: track 17.9 -> 16.2 mm
- net /DEBUG_RX_MCU: track 18.3 -> 17.0 mm
- net /DEBUG_TX_MCU: track 18.8 -> 17.9 mm
- net /VDD: track 74.4 -> 74.6 mm, vias 2 -> 1

Commit message: Minor updates
Parts:
- moved C13 8.02 mm to (198.4, -12.7)
- moved C12 8.00 mm to (198.4, -16.1)
- moved Y1 7.41 mm to (203.5, -16.0)
- moved C15 5.84 mm to (198.6, -29.5)
- moved Y2 5.84 mm to (201.4, -27.4)
- moved C14 5.84 mm to (198.6, -27.4)
- turned C7 to 90 degrees
- turned D3 to 0 degrees
- turned D4 to 0 degrees
- turned R4 to 270 degrees
- turned R5 to 270 degrees
Connections:
- D3 pad 1: GND -> Net-(D3-Pad1)
- D3 pad 2: Net-(D3-Pad2) -> /VDDS
- D4 pad 1: GND -> Net-(D4-Pad1)
- D4 pad 2: Net-(D4-Pad2) -> /VDDS
- F1 pad 1: Net-(F1-Pad1) -> /VBUS
- R4 pad 1: /LED1_MCU -> Net-(D3-Pad1)
- R4 pad 2: Net-(D3-Pad2) -> /LED1_MCU
- R5 pad 1: /LED2_MCU -> Net-(D4-Pad1)
- R5 pad 2: Net-(D4-Pad2) -> /LED2_MCU
- RV1 pad 1: /VBUS -> GND1
- RV1 pad 2: Net-(F1-Pad1) -> /VBUS
Routing:
- net /VDDS: track 45.8 -> 64.8 mm
- net GND1: track 31.4 -> 43.9 mm
- net /X48M_N: track 29.1 -> 21.0 mm
- net /X48M_P: track 26.6 -> 19.0 mm
- net /X32K_P: track 17.2 -> 11.3 mm
- net /X32K_N: track 17.2 -> 11.3 mm
- net Net-(D3-Pad2): track 4.99 -> 0.00 mm
- net Net-(D3-Pad1): track 0.00 -> 4.99 mm
- net Net-(D4-Pad2): track 4.78 -> 0.00 mm
- net Net-(D4-Pad1): track 0.00 -> 4.78 mm
- net Net-(F1-Pad1): track 1.71 -> 0.00 mm
- net /VBUS: track 7.04 -> 8.35 mm
- net GND: track 2.84 -> 3.20 mm, vias 546 -> 540
- net (no net): vias 0 -> 1
